File: pcb/PT2258-S_Breakout.sch (EAGLE design)
At the start: 37 parts, among them U1 PT2258-S, X1 INPUT, X2 I2C, X3 POWER, X4 OUTPUT

Commit message: Fix SOP-20-300 footprint
Parts:
- U1: device M2M-IC:PT2258 -> M2M-IC:PT2258-S
Changed lines of the file:
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@@
 <parts>
 <part name="FRAME1" library="M2M-Frames" deviceset="FRAME-M2M-A4L" device=""/>
-<part name="U1" library="M2M-IC" deviceset="PT2258" device="" value="PT2258-S"/>
+<part name="U1" library="M2M-IC" deviceset="PT2258" device="-S" value="PT2258-S"/>
 <part name="SUPPLY1" library="M2M-Power" deviceset="VCC" device=""/>
 <part name="SUPPLY2" library="M2M-Power" deviceset="AGND" device=""/>
